File: electronics/foxy/foxy.kicad_sch (KiCad schematic)
At the start: 13 parts, among them J1 SMA, J2 Conn_01x07_Pin, J3 Conn_alim

Commit message: add function blocs in schema
Other:
- note added: "Low Pass Filter"
- note added: "Power supply"
- note added: "SI5351"
Changed lines of the file:
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@@
+		)
+	)
+	(rectangle
+		(start 90.17 111.76)
+		(end 115.57 148.59)
+		(stroke
+			(width 0)
+			(type default)
+		)
+		(fill
+			(type none)
+		)
+	)
+	(rectangle
+		(start 161.29 133.35)
+		(end 222.25 163.83)
+		(stroke
+			(width 0)
+			(type default)
+		)
+		(fill
+			(type none)
+		)
+	)
+	(rectangle
+		(start 80.01 39.37)
+		(end 110.49 77.47)
+		(stroke
+			(width 0)
+			(type default)
+		)
+		(fill
+			(type none)
+		)
+	)
+	(text "SI5351"
+		(exclude_from_sim no)
+		(at 94.996 114.3 0)
+		(effects
+			(font
+				(size 1.27 1.27)
+			)
+		)
+	)
+	(text "Low Pass Filter\n"
+		(exclude_from_sim no)
+		(at 169.418 135.636 0)
+		(effects
+			(font
+				(size 1.27 1.27)
+			)
+		)
+	)
+	(text "Power supply"
+		(exclude_from_sim no)
+		(at 87.63 42.418 0)
+		(effects
+			(font
+				(size 1.27 1.27)
+			)
 		)
 	)
